File: 100base-t1-converter.kicad_pcb (KiCad board)
At the start: 4 copper layers, 87.6 x 50.8 mm, 83 parts, among them J1 Conn_01x02, J2 Conn_01x03, J3 Conn_01x03, J4 Conn_01x02, J5 8P8C_LED_Shielded, J6 USB_B_Micro, U1 AP1117-33, U2 TJA1101, U3 blue_pill, U4 SR8201F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

Commit message: JPWORK modify commit
Parts:
- FB2, FB4: value 120R -> 0
Connections:
- net /micro/~INT renamed /micro/~{INT}
- net /tx_mac/RXC renamed /tja1101/TXC
- net /tx_mac/RXD0 renamed /tja1101/TXD0
- net /tx_mac/RXD1 renamed /tja1101/TXD1
- net /tx_mac/RXD2 renamed /tja1101/TXD2
- net /tx_mac/RXD3 renamed /tja1101/TXD3
- net /tx_mac/RXDV renamed /tja1101/TXEN
- net /tx_mac/RXER renamed /tja1101/TXER
- C10 pad 2: Net-(C10-Pad2) -> (no net)
- C17 pad 1: Net-(C17-Pad1) -> unconnected-(C17-Pad1)
- C19 pad 2: Net-(C19-Pad2) -> unconnected-(C19-Pad2)
- C20 pad 2: Net-(C20-Pad2) -> unconnected-(C20-Pad2)
- C4 pad 2: Net-(C4-Pad2) -> unconnected-(#FLG0104-pwr-Pad1)
- C5 pad 2: Net-(C5-Pad2) -> unconnected-(#FLG0105-pwr-Pad1)
- C7 pad 2: Net-(C4-Pad2) -> unconnected-(#FLG0104-pwr-Pad1)
- C8 pad 1: Net-(C4-Pad2) -> unconnected-(#FLG0104-pwr-Pad1)
- C9 pad 2: Net-(C10-Pad2) -> (no net)
- FB1 pad 1: Net-(C5-Pad2) -> unconnected-(#FLG0105-pwr-Pad1)
- FB3 pad 1: Net-(C4-Pad2) -> unconnected-(#FLG0104-pwr-Pad1)
- J2 pad 2: Net-(J2-Pad2) -> (no net)
- J3 pad 2: Net-(J3-Pad2) -> (no net)
- J4 pad 1: Net-(J4-Pad1) -> unconnected-(#FLG0106-pwr-Pad1)
- J5 pad 10: Net-(J5-Pad10) -> unconnected-(R23-Pad2)
- J5 pad 11: Net-(J5-Pad11) -> unconnected-(R21-Pad2)
- J5 pad 4: Net-(C19-Pad2) -> unconnected-(C19-Pad2)
- J5 pad 5: Net-(C20-Pad2) -> unconnected-(C20-Pad2)
- J5 pad 7: Net-(J5-Pad7) -> (no net)
- J6 pad 2: Net-(J6-Pad2) -> unconnected-(J6-D--Pad2)
- J6 pad 3: Net-(J6-Pad3) -> unconnected-(J6-D+-Pad3)
- J6 pad 4: Net-(J6-Pad4) -> unconnected-(J6-ID-Pad4)
- R13 pad 1: Net-(R13-Pad1) -> (no net)
- R14 pad 1: Net-(R14-Pad1) -> (no net)
- R15 pad 1: Net-(R15-Pad1) -> (no net)
- R16 pad 2: Net-(R15-Pad1) -> (no net)
- R18 pad 2: Net-(C17-Pad1) -> unconnected-(C17-Pad1)
- R19 pad 1: Net-(C17-Pad1) -> unconnected-(C17-Pad1)
- R20 pad 1: Net-(C17-Pad1) -> unconnected-(C17-Pad1)
- R21 pad 2: Net-(J5-Pad11) -> unconnected-(R21-Pad2)
- R23 pad 2: Net-(J5-Pad10) -> unconnected-(R23-Pad2)
- R3 pad 1: Net-(J2-Pad2) -> (no net)
- R6 pad 1: Net-(J3-Pad2) -> (no net)
- R9 pad 1: Net-(R9-Pad1) -> (no net)
- RN1 pad 5: Net-(RN1-Pad5) -> (no net)
- RN1 pad 6: Net-(RN1-Pad6) -> (no net)
- RN1 pad 7: Net-(RN1-Pad7) -> (no net)
- RN1 pad 8: Net-(RN1-Pad8) -> (no net)
- RN2 pad 1: Net-(RN2-Pad1) -> unconnected-(U4-RXD[0]-Pad9)
- RN2 pad 2: Net-(RN2-Pad2) -> unconnected-(U4-RXD[1]-Pad10)
- RN2 pad 3: Net-(RN2-Pad3) -> unconnected-(U4-RXD[2]/INTB-Pad11)
- RN2 pad 4: Net-(RN2-Pad4) -> unconnected-(U4-RXD[3]/CLK_CTL-Pad12)
- U2 pad 16: Net-(C10-Pad2) -> (no net)
- U2 pad 17: Net-(R14-Pad1) -> (no net)
- U2 pad 18: Net-(R13-Pad1) -> (no net)
- U2 pad 19: Net-(C4-Pad2) -> unconnected-(#FLG0104-pwr-Pad1)
- U2 pad 21: Net-(RN1-Pad5) -> (no net)
- U2 pad 22: Net-(RN1-Pad6) -> (no net)
- U2 pad 23: Net-(RN1-Pad7) -> (no net)
- U2 pad 24: Net-(RN1-Pad8) -> (no net)
- U2 pad 27: Net-(C4-Pad2) -> unconnected-(#FLG0104-pwr-Pad1)
- U2 pad 35: Net-(R9-Pad1) -> (no net)
- U2 pad 4: Net-(R15-Pad1) -> (no net)
- U2 pad 9: Net-(C5-Pad2) -> unconnected-(#FLG0105-pwr-Pad1)
- U3 pad 1: Net-(U3-Pad1) -> (no net)
- U3 pad 10: Net-(U3-Pad10) -> (no net)
- U3 pad 16: Net-(U3-Pad16) -> (no net)
- U3 pad 17: Net-(U3-Pad17) -> (no net)
- U3 pad 18: Net-(J4-Pad1) -> unconnected-(#FLG0106-pwr-Pad1)
- U3 pad 2: Net-(U3-Pad2) -> (no net)
- U3 pad 20: Net-(U3-Pad20) -> (no net)
- U3 pad 21: Net-(U3-Pad21) -> (no net)
- U3 pad 22: Net-(U3-Pad22) -> (no net)
- U3 pad 23: Net-(U3-Pad23) -> (no net)
- U3 pad 24: Net-(U3-Pad24) -> (no net)
- U3 pad 25: Net-(U3-Pad25) -> (no net)
- U3 pad 26: Net-(U3-Pad26) -> (no net)
- U3 pad 27: Net-(U3-Pad27) -> (no net)
- U3 pad 28: Net-(U3-Pad28) -> (no net)
- U3 pad 29: Net-(U3-Pad29) -> (no net)
- U3 pad 3: Net-(U3-Pad3) -> (no net)
- U3 pad 30: Net-(U3-Pad30) -> (no net)
- U3 pad 31: Net-(U3-Pad31) -> (no net)
- U3 pad 32: Net-(U3-Pad32) -> (no net)
- U3 pad 33: Net-(U3-Pad33) -> (no net)
- U3 pad 34: Net-(U3-Pad34) -> (no net)
- U3 pad 35: Net-(U3-Pad35) -> (no net)
- U3 pad 36: Net-(U3-Pad36) -> (no net)
- U3 pad 37: Net-(U3-Pad37) -> (no net)
- U3 pad 38: Net-(U3-Pad38) -> (no net)
- U3 pad 4: Net-(U3-Pad4) -> (no net)
- U3 pad 5: Net-(U3-Pad5) -> (no net)
- U3 pad 6: Net-(U3-Pad6) -> (no net)
- U3 pad 7: Net-(U3-Pad7) -> (no net)
- U3 pad 8: Net-(U3-Pad8) -> (no net)
- U3 pad 9: Net-(U3-Pad9) -> (no net)
- U4 pad 10: Net-(RN2-Pad2) -> unconnected-(U4-RXD[1]-Pad10)
- U4 pad 11: Net-(RN2-Pad3) -> unconnected-(U4-RXD[2]/INTB-Pad11)
- U4 pad 12: Net-(RN2-Pad4) -> unconnected-(U4-RXD[3]/CLK_CTL-Pad12)
- U4 pad 9: Net-(RN2-Pad1) -> unconnected-(U4-RXD[0]-Pad9)
Routing:
- net (no net): track 0.00 -> 81.9 mm, vias 0 -> 2
- net unconnected-(#FLG0106-pwr-Pad1): track 0.00 -> 21.0 mm
- net Net-(J4-Pad1): track 21.0 -> 0.00 mm
- net Net-(J2-Pad2): track 19.8 -> 0.00 mm
- net unconnected-(C17-Pad1): track 0.00 -> 16.0 mm
- net Net-(C17-Pad1): track 16.0 -> 0.00 mm
- net unconnected-(#FLG0104-pwr-Pad1): track 0.00 -> 15.3 mm, vias 0 -> 2
- net Net-(C4-Pad2): track 15.3 -> 0.00 mm, vias 2 -> 0
- net Net-(J3-Pad2): track 14.2 -> 0.00 mm
- net Net-(R13-Pad1): track 11.8 -> 0.00 mm, vias 2 -> 0
- net unconnected-(U4-RXD[0]-Pad9): track 0.00 -> 9.21 mm
- net Net-(RN2-Pad1): track 9.21 -> 0.00 mm
- net Net-(R15-Pad1): track 9.14 -> 0.00 mm
- net unconnected-(C20-Pad2): track 0.00 -> 8.59 mm
- net Net-(C20-Pad2): track 8.59 -> 0.00 mm
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Other:
- net class Default removed
- board text added: "100Base-TX to 100Base-T1 Converter for Education Copyright JP WORKS 2025 Licensed CC-BY-SA https://github.com/TLDSJPWORK/100base-t1-converter Rev 1.0"
- board text removed: "100Base-TX to 100Base-T1 Converter Copyright Mitchell Johnson 2019 Licensed CC-BY-SA https://github.com/ehntoo/100base-t1-converter Rev 0.1"
